File: STM32U5G9ZJTx.kicad_sch (KiCad schematic)
At the start: 42 parts, among them J1 Conn_ST_STDC14, SW1 SW_Push, SW2 SW_Push, U1 STM32U5G9ZJTxQ, Y1 16MHz, Y2 32.768KHz

Commit message: Change bypass capacitor to 0201
Parts:
- C1, C10, C11, C14, C16, C18, C19, C2, C20, C21, C23, C24, C25, C26, C3, C33, C4, C5, C6, C7, C8, C9: footprint Capacitor_SMD:C_0402_1005Metric -> Capacitor_SMD:C_0201_0603Metric
- C17, C22, C27, C28: footprint Capacitor_SMD:C_0603_1608Metric -> Capacitor_SMD:C_0402_1005Metric
Changed lines of the file:
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@@
 		(polyline
 			(pts
-				(xy 304.8 144.78) (xy 304.8 119.38) (xy 274.32 119.38) (xy 274.32 144.78)
+				(xy 313.69 119.38) (xy 313.69 144.78) (xy 360.68 144.78) (xy 360.68 119.38)
 			)
 			(stroke
@@
 		(polyline
 			(pts
-				(xy 313.69 110.49) (xy 349.25 110.49) (xy 349.25 85.09) (xy 313.69 85.09)
+				(xy 364.49 119.38) (xy 364.49 144.78) (xy 400.05 144.78) (xy 400.05 119.38)
 			)
 			(stroke
@@
 		(polyline
 			(pts
-				(xy 364.49 119.38) (xy 364.49 144.78) (xy 400.05 144.78) (xy 400.05 119.38)
+				(xy 358.14 110.49) (xy 386.08 110.49) (xy 386.08 85.09) (xy 358.14 85.09)
 			)
 			(stroke
@@
 		(polyline
 			(pts
-				(xy 274.32 110.49) (xy 304.8 110.49) (xy 304.8 85.09) (xy 274.32 85.09)
+				(xy 304.8 144.78) (xy 304.8 119.38) (xy 274.32 119.38) (xy 274.32 144.78)
 			)
 			(stroke
@@
 		(polyline
 			(pts
-				(xy 240.03 78.74) (xy 381 78.74) (xy 381 52.07) (xy 240.03 52.07)
+				(xy 240.03 154.94) (xy 285.75 154.94) (xy 285.75 186.69) (xy 240.03 186.69)
 			)
 			(stroke
@@
 		(polyline
 			(pts
-				(xy 240.03 44.45) (xy 276.86 44.45) (xy 276.86 16.51) (xy 240.03 16.51)
+				(xy 313.69 110.49) (xy 349.25 110.49) (xy 349.25 85.09) (xy 313.69 85.09)
 			)
 			(stroke
@@
 		(polyline
 			(pts
-				(xy 240.03 144.78) (xy 265.43 144.78) (xy 265.43 119.38) (xy 240.03 119.38)
+				(xy 240.03 44.45) (xy 276.86 44.45) (xy 276.86 16.51) (xy 240.03 16.51)
 			)
 			(stroke
@@
 		(polyline
 			(pts
-				(xy 240.03 154.94) (xy 285.75 154.94) (xy 285.75 186.69) (xy 240.03 186.69)
+				(xy 240.03 78.74) (xy 381 78.74) (xy 381 52.07) (xy 240.03 52.07)
 			)
 			(stroke
@@
 		(polyline
 			(pts
-				(xy 358.14 110.49) (xy 386.08 110.49) (xy 386.08 85.09) (xy 358.14 85.09)
+				(xy 240.03 144.78) (xy 265.43 144.78) (xy 265.43 119.38) (xy 240.03 119.38)
 			)
 			(stroke
@@
 		(polyline
 			(pts
-				(xy 313.69 119.38) (xy 313.69 144.78) (xy 360.68 144.78) (xy 360.68 119.38)
+				(xy 274.32 110.49) (xy 304.8 110.49) (xy 304.8 85.09) (xy 274.32 85.09)
 			)
 			(stroke
@@
 			)
 		)
-		(property "Footprint" "Capacitor_SMD:C_0402_1005Metric"
+		(property "Footprint" "Capacitor_SMD:C_0201_0603Metric"
 			(at 256.54 132.08 0)
 			(effects
@@
 			)
 		)
-		(property "Footprint" "Capacitor_SMD:C_0603_1608Metric"
+		(property "Footprint" "Capacitor_SMD:C_0402_1005Metric"
 			(at 338.7852 137.16 0)
 			(effects
@@
 			)
 		)
-		(property "Footprint" "Capacitor_SMD:C_0402_1005Metric"
+		(property "Footprint" "Capacitor_SMD:C_0201_0603Metric"
 			(at 279.4 66.04 0)
 			(effects
@@
 			)
 		)
-		(property "Footprint" "Capacitor_SMD:C_0402_1005Metric"
+		(property "Footprint" "Capacitor_SMD:C_0201_0603Metric"
 			(at 267.97 31.75 0)
 			(effects
@@
 			)
 		)
-		(property "Footprint" "Capacitor_SMD:C_0603_1608Metric"
+		(property "Footprint" "Capacitor_SMD:C_0402_1005Metric"
 			(at 351.4852 137.16 0)
 			(effects
@@
 			)
 		)
-		(property "Footprint" "Capacitor_SMD:C_0402_1005Metric"
+		(property "Footprint" "Capacitor_SMD:C_0201_0603Metric"
 			(at 306.07 212.09 0)
 			(effects
@@
 			)
 		)
-		(property "Footprint" "Capacitor_SMD:C_0402_1005Metric"
+		(property "Footprint" "Capacitor_SMD:C_0201_0603Metric"
 			(at 302.26 66.04 0)
 			(effects
@@
 			)
 		)
-		(property "Footprint" "Capacitor_SMD:C_0402_1005Metric"
+		(property "Footprint" "Capacitor_SMD:C_0201_0603Metric"
 			(at 336.55 66.04 0)
 			(effects
@@
 			)
 		)
-		(property "Footprint" "Capacitor_SMD:C_0402_1005Metric"
+		(property "Footprint" "Capacitor_SMD:C_0201_0603Metric"
 			(at 382.27 133.35 0)
 			(effects
@@
 			)
 		)
-		(property "Footprint" "Capacitor_SMD:C_0402_1005Metric"
+		(property "Footprint" "Capacitor_SMD:C_0201_0603Metric"
 			(at 290.83 66.04 0)
 			(effects
@@
 			)
 		)
-		(property "Footprint" "Capacitor_SMD:C_0402_1005Metric"
+		(property "Footprint" "Capacitor_SMD:C_0201_0603Metric"
 			(at 313.69 66.04 0)
 			(effects
@@
 			)
 		)
-		(property "Footprint" "Capacitor_SMD:C_0603_1608Metric"
+		(property "Footprint" "Capacitor_SMD:C_0402_1005Metric"
 			(at 280.3652 137.16 0)
 			(effects
@@
 			)
 		)
-		(property "Footprint" "Capacitor_SMD:C_0402_1005Metric"
+		(property "Footprint" "Capacitor_SMD:C_0201_0603Metric"
 			(at 347.98 66.04 0)
 			(effects
@@
 			)
 		)
-		(property "Footprint" "Capacitor_SMD:C_0402_1005Metric"
+		(property "Footprint" "Capacitor_SMD:C_0201_0603Metric"
 			(at 256.54 66.04 0)
 			(effects
@@
 			)
 		)
-		(property "Footprint" "Capacitor_SMD:C_0402_1005Metric"
+		(property "Footprint" "Capacitor_SMD:C_0201_0603Metric"
 			(at 245.11 97.79 0)
 			(effects
@@
 			)
 		)
-		(property "Footprint" "Capacitor_SMD:C_0402_1005Metric"
+		(property "Footprint" "Capacitor_SMD:C_0201_0603Metric"
 			(at 370.84 133.35 0)
 			(effects
@@
 			)
 		)
-		(property "Footprint" "Capacitor_SMD:C_0402_1005Metric"
+		(property "Footprint" "Capacitor_SMD:C_0201_0603Metric"
 			(at 290.83 133.35 0)
 			(effects
@@
 			)
 		)
-		(property "Footprint" "Capacitor_SMD:C_0402_1005Metric"
+		(property "Footprint" "Capacitor_SMD:C_0201_0603Metric"
 			(at 256.54 31.75 0)
 			(effects
@@
 			)
 		)
-		(property "Footprint" "Capacitor_SMD:C_0402_1005Metric"
+		(property "Footprint" "Capacitor_SMD:C_0201_0603Metric"
 			(at 331.47 97.79 0)
 			(effects
@@
 			)
 		)
-		(property "Footprint" "Capacitor_SMD:C_0402_1005Metric"
+		(property "Footprint" "Capacitor_SMD:C_0201_0603Metric"
 			(at 267.97 66.04 0)
 			(effects
@@
 			)
 		)
-		(property "Footprint" "Capacitor_SMD:C_0402_1005Metric"
+		(property "Footprint" "Capacitor_SMD:C_0201_0603Metric"
 			(at 359.41 66.04 0)
 			(effects
@@
 			)
 		)
-		(property "Footprint" "Capacitor_SMD:C_0402_1005Metric"
+		(property "Footprint" "Capacitor_SMD:C_0201_0603Metric"
 			(at 325.12 66.04 0)
 			(effects
@@
 			)
 		)
-		(property "Footprint" "Capacitor_SMD:C_0402_1005Metric"
+		(property "Footprint" "Capacitor_SMD:C_0201_0603Metric"
 			(at 363.22 97.79 0)
 			(effects
@@
 			)
 		)
-		(property "Footprint" "Capacitor_SMD:C_0402_1005Metric"
+		(property "Footprint" "Capacitor_SMD:C_0201_0603Metric"
 			(at 370.84 66.04 0)
 			(effects
@@
 			)
 		)
-		(property "Footprint" "Capacitor_SMD:C_0402_1005Metric"
+		(property "Footprint" "Capacitor_SMD:C_0201_0603Metric"
 			(at 279.4 97.79 0)
 			(effects
@@
 			)
 		)
-		(property "Footprint" "Capacitor_SMD:C_0603_1608Metric"
+		(property "Footprint" "Capacitor_SMD:C_0402_1005Metric"
 			(at 246.0752 135.89 0)
 			(effects
